File: PCB/raspi_foundation_files/LLAMABELL.kicad_sch (KiCad schematic)
At the start: 20 parts, among them J1 Conn_01x03, J2 Conn_02x07_Odd_Even, J3 Conn_01x03, J9 THD-02-R, U1 TPD4EUSB30, U2 TPD4EUSB30, U3 MagJack-A70-112-331N126, U5 74LVC1G07SE-7, U9 74LVC1G07SE-7

Commit message: Who_the_fuck_knows.jpg
Parts:
- removed C1: 100n, Capacitor_SMD:C_0402_1005Metric, symbol Device:C
- removed D1: LED Red, LED_SMD:LED_0603_1608Metric, symbol Device:LED
- removed J1, J3: Conn_01x03, Connector_PinHeader_2.54mm:PinHeader_1x03_P2.54mm_Vertical, symbol Connector_Generic:Conn_01x03
- removed J9: THD-02-R, Connector_PinHeader_2.54mm:PinHeader_2x02_P2.54mm_Vertical, symbol Connector_Generic:Conn_02x02_Odd_Even
- removed R10: 1k, Resistor_SMD:R_0402_1005Metric, symbol Device:R
- removed R2, R3: 470R, Resistor_SMD:R_0402_1005Metric, symbol Device:R
- removed TP5: TestPoint, TestPoint:TestPoint_Pad_2.0x2.0mm, symbol Connector:TestPoint
- removed U1, U2: TPD4EUSB30, Package_SON:USON-10_2.5x1.0mm_P0.5mm, symbol CM4IO:TPD4EUSB30
- removed U3: MagJack-A70-112-331N126, CM4IO:TRJG0926HENL, symbol CM4IO:MagJack-A70-112-331N126
- removed U5: 74LVC1G07SE-7, Package_TO_SOT_SMD:SOT-353_SC-70-5, symbol CM4IO:74LVC1G07_copy
Connections:
- net WL_nDis: no longer names the net of Module1.89 (WL_nDisable)
Other:
- note removed: "Ethernet"
- note removed: "Ethernet POE Protection"
- note removed: "Not Fitted headers"
- note removed: "POE Header"
- note removed: "PWR LED"
